Commit message: Fixed Fingers

File: urdf/gripbot_2.urdf (robot description, URDF)
Before this commit: robot gripbot, 18 links, 17 joints
Links:
- link finger_1_base_link: mass 0.1010 -> 0.01308
- link finger_1_distal_link: mass 0.101 -> 0.01681805
- link finger_1_mid_link: mass 0.101 -> 0.01317208; geometry collision box size=0.01784 0.01899 0.03309; visual mesh filename=package://gripbot_description/meshes/stl/FingerMid.001.stl scale=1.0 1.0 1.0
- link finger_1_proximal_link: mass 0.101 -> 0.01907932
- link finger_2_base_link: mass 0.101 -> 0.01308
- link finger_2_distal_link: mass 0.101 -> 0.01681805
- link finger_2_mid_link: mass 0.101 -> 0.01317208; geometry collision box size=0.01784 0.01899 0.03281; visual mesh filename=package://gripbot_description/meshes/stl/FingerMid.002.stl scale=1.0 1.0 1.0
- link finger_2_proximal_link: mass 0.101 -> 0.01907932
- link finger_3_distal_link: mass 0.101 -> 0.01681805; geometry collision box size=0.0175 0.02023 0.04043; visual mesh filename=package://gripbot_description/meshes/stl/FingerDistal.003.s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 scale=1.0 1.0 1.0
- link finger_3_mid_link: mass 0.101 -> 0.01317208; geometry collision box size=0.01784 0.01899 0.03281; visual mesh filename=package://gripbot_description/meshes/stl/FingerMid.003.stl scale=1.0 1.0 1.0
- link finger_3_proximal_link: mass 0.101 -> 0.01907932
Joints:
- joint arm_visual_link: limit lower=-1.5708 upper=0.59341 effort=135.0 velocity=6.28319 -> lower=-1.5708 upper=0.59341 effort=135.0 velocity=1.0
- joint base_column_link: limit lower=-3.14159 upper=3.14159 effort=135.0 velocity=6.28319 -> lower=-3.14159 upper=3.14159 effort=135.0 velocity=1.0
- joint base_wrist_link: limit lower=-1.5708 upper=1.5708 effort=10000.0 velocity=6.00 -> lower=-1.5708 upper=1.5708 effort=10000.0 velocity=1.0
- joint finger_1_base_link: limit lower=-2.04204 upper=0.7854 effort=10000.0 velocity=60000 -> lower=-2.04204 upper=0.7854 effort=10000.0 velocity=1.0
- joint finger_1_distal_link: limit lower=0 upper=1.5708 effort=10000.0 velocity=60000 -> lower=0 upper=1.5708 effort=10000.0 velocity=1.0
- joint finger_1_mid_link: limit lower=0 upper=1.5708 effort=10000.0 velocity=60000 -> lower=0 upper=1.5708 effort=10000.0 velocity=1.0
- joint finger_1_proximal_link: limit lower=0 upper=1.5708 effort=10000.0 velocity=60000 -> lower=0 upper=1.5708 effort=10000.0 velocity=1.0
- joint finger_2_base_link: limit lower=-0.7854 upper=2.04204 effort=10000.0 velocity=60000 -> lower=-0.7854 upper=2.04204 effort=10000.0 velocity=1.0
- joint finger_2_distal_link: limit lower=-1.5708 upper=0 effort=10000.0 velocity=60000 -> lower=-1.5708 upper=0 effort=10000.0 velocity=1.0
- joint finger_2_mid_link: limit lower=-1.5708 upper=0 effort=10000.0 velocity=60000 -> lower=-1.5708 upper=0 effort=10000.0 velocity=1.0
- joint finger_2_proximal_link: limit lower=-1.5708 upper=0 effort=10000.0 velocity=60000 -> lower=-1.5708 upper=0 effort=10000.0 velocity=1.0
- joint finger_3_distal_link: limit lower=0 upper=1.72788 effort=10000.0 velocity=60000 -> lower=0 upper=1.72788 effort=10000.0 velocity=1.0
- joint finger_3_mid_link: limit lower=0 upper=1.72788 effort=10000.0 velocity=60000 -> lower=0 upper=1.72788 effort=10000.0 velocity=1.0
- joint finger_3_proximal_link: limit lower=-0.7854 upper=1.72788 effort=10000.0 velocity=60000 -> lower=-0.7854 upper=1.72788 effort=10000.0 velocity=1.0
- joint forearm_visual_link: limit lower=-1.5708 upper=2.18166 effort=135.0 velocity=60000.28319 -> lower=-1.5708 upper=2.18166 effort=135.0 velocity=1.0
- joint girdle_visual_link: limit lower=-0.5236 upper=1.95477 effort=50000.0 velocity=6000.0 -> lower=-0.5236 upper=1.95477 effort=50000.0 velocity=1.0
